File: Circuits/Boards/MotorControllerBoard/MainBoard/MainBoard.sch (EAGLE design)
At the start: 56 parts, among them IC2 788TV, M1 IRFS7537PBF, M2 IRFS7537PBF, M3 IRFS7537PBF, M4 IRFS7537PBF, Q1 2N3904, Q2 2N3904, Q3 2N3904, Q4 2N3904, Q5 2N3904, Q6 2N3904, Q7 2N3904, Q8 2N3904

Commit message: Finished board files and updated gitignore
Parts:
- added PAD8, PAD9: WIREPAD2,54/1,1, wirepad:WIREPAD2,54/1,1
- PAD2: value WIREPAD4,16O1,6 -> (none); device wirepad:WIREPAD4,16O1,6 -> wirepad:3,81/1,4
- PAD4: value (none) -> WIREPAD4,16O1,6; device wirepad:2,54/1,0 -> wirepad:WIREPAD4,16O1,6
- PAD6: device wirepad:3,81/1,4 -> wirepad:2,54/1,0
Connections:
- new net FBJ: PAD9.P, Q7.B
- net FB: now also PAD8.P; no longer Q7.B
- net MN: now also PAD4.P; no longer PAD3.P
- net MP: now also PAD3.P; no longer PAD2.P
- net N$1: now also PAD2.P; no longer PAD6.P
- net PWM: now also PAD6.P; no longer PAD4.P
Other:
- moved on the sheet: PAD1, PAD3, PAD5
Changed lines of the file:
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@@
 <part name="C4" library="rcl" library_urn="urn:adsk.eagle:library:334" deviceset="CPOL-US" device="E2.5-7" package3d_urn="urn:adsk.eagle:package:23345/1"/>
 <part name="C5" library="rcl" library_urn="urn:adsk.eagle:library:334" deviceset="CPOL-US" device="E2.5-7" package3d_urn="urn:adsk.eagle:package:23345/1"/>
-<part name="PAD2" library="wirepad" library_urn="urn:adsk.eagle:library:412" deviceset="WIREPAD" device="4,16O1,6" package3d_urn="urn:adsk.eagle:package:30843/1" value="WIREPAD4,16O1,6"/>
 <part name="PAD3" library="wirepad" library_urn="urn:adsk.eagle:library:412" deviceset="WIREPAD" device="4,16O1,6" package3d_urn="urn:adsk.eagle:package:30843/1" value="WIREPAD4,16O1,6"/>
-<part name="PAD4" library="wirepad" library_urn="urn:adsk.eagle:library:412" deviceset="2,54/1,0" device="" package3d_urn="urn:adsk.eagle:package:30828/1"/>
-<part name="PAD5" library="wirepad" library_urn="urn:adsk.eagle:library:412" deviceset="3,81/1,4" device="" package3d_urn="urn:adsk.eagle:package:30835/1"/>
-<part name="PAD6" library="wirepad" library_urn="urn:adsk.eagle:library:412" deviceset="3,81/1,4" device="" package3d_urn="urn:adsk.eagle:package:30835/1"/>
+<part name="PAD4" library="wirepad" library_urn="urn:adsk.eagle:library:412" deviceset="WIREPAD" device="4,16O1,6" package3d_urn="urn:adsk.eagle:package:30843/1" value="WIREPAD4,16O1,6"/>
+<part name="PAD6" library="wirepad" library_urn="urn:adsk.eagle:library:412" deviceset="2,54/1,0" device="" package3d_urn="urn:adsk.eagle:package:30828/1"/>
+<part name="PAD1" library="wirepad" library_urn="urn:adsk.eagle:library:412" deviceset="3,81/1,4" device="" package3d_urn="urn:adsk.eagle:package:30835/1"/>
+<part name="PAD2" library="wirepad" library_urn="urn:adsk.eagle:library:412" deviceset="3,81/1,4" device="" package3d_urn="urn:adsk.eagle:package:30835/1"/>
 <part name="PAD7" library="wirepad" library_urn="urn:adsk.eagle:library:412" deviceset="2,54/1,0" device="" package3d_urn="urn:adsk.eagle:package:30828/1"/>
 <part name="R19" library="ptc-ntc" library_urn="urn:adsk.eagle:library:332" deviceset="PTC660A" device="" package3d_urn="urn:adsk.eagle:package:22777/1"/>
@@
 <part name="R22" library="ptc-ntc" library_urn="urn:adsk.eagle:library:332" deviceset="PTC660A" device="" package3d_urn="urn:adsk.eagle:package:22777/1"/>
 <part name="R23" library="ptc-ntc" library_urn="urn:adsk.eagle:library:332" deviceset="PTC660A" device="" package3d_urn="urn:adsk.eagle:package:22777/1"/>
-<part name="PAD1" library="wirepad" library_urn="urn:adsk.eagle:library:412" deviceset="3,81/1,4" device="" package3d_urn="urn:adsk.eagle:package:30835/1"/>
+<part name="PAD5" library="wirepad" library_urn="urn:adsk.eagle:library:412" deviceset="3,81/1,4" device="" package3d_urn="urn:adsk.eagle:package:30835/1"/>
+<part name="PAD8" library="wirepad" library_urn="urn:adsk.eagle:library:412" deviceset="WIREPAD" device="2,54/1,1" package3d_urn="urn:adsk.eagle:package:30836/1"/>
+<part name="PAD9" library="wirepad" library_urn="urn:adsk.eagle:library:412" deviceset="WIREPAD" device="2,54/1,1" package3d_urn="urn:adsk.eagle:package:30836/1"/>
 </parts>
 <sheets>
@@
 <instance part="C4" gate="G$1" x="-88.9" y="30.48"/>
 <instance part="C5" gate="G$1" x="-127" y="30.48"/>
-<instance part="PAD2" gate="G$1" x="101.6" y="109.22" rot="R180"/>
-<instance part="PAD3" gate="G$1" x="114.3" y="109.22"/>
-<instance part="PAD4" gate="P" x="109.22" y="5.08" rot="R90"/>
-<instance part="PAD5" gate="1" x="175.26" y="50.8" rot="R180"/>
-<instance part="PAD6" gate="1" x="109.22" y="160.02" rot="R270"/>
+<instance part="PAD3" gate="G$1" x="101.6" y="109.22" rot="R180"/>
+<instance part="PAD4" gate="G$1" x="114.3" y="109.22"/>
+<instance part="PAD6" gate="P" x="109.22" y="5.08" rot="R90"/>
+<instance part="PAD1" gate="1" x="175.26" y="50.8" rot="R180"/>
+<instance part="PAD2" gate="1" x="109.22" y="160.02" rot="R270"/>
 <instance part="PAD7" gate="P" x="-50.8" y="142.24" rot="R270"/>
 <instance part="R19" gate="1" x="88.9" y="149.86" rot="R180"/>
@@
 <instance part="R22" gate="1" x="119.38" y="149.86" rot="R180"/>
 <instance part="R23" gate="1" x="129.54" y="149.86" rot="R180"/>
-<instance part="PAD1" gate="1" x="53.34" y="43.18" rot="R90"/>
+<instance part="PAD5" gate="1" x="167.64" y="43.18" rot="R90"/>
+<instance part="PAD8" gate="G$1" x="-17.78" y="129.54"/>
+<instance part="PAD9" gate="G$1" x="177.8" y="68.58" rot="R180"/>
 </instances>
 <busses>
@@
 <junction x="93.98" y="109.22"/>
 <wire x1="99.06" y1="109.22" x2="93.98" y2="109.22" width="0.1524" layer="91"/>
-<pinref part="PAD2" gate="G$1" pin="P"/>
+<pinref part="PAD3" gate="G$1" pin="P"/>
 </segment>
 </net>
@@
 <wire x1="134.62" y1="109.22" x2="134.62" y2="101.6" width="0.1524" layer="91"/>
 <junction x="134.62" y="109.22"/>
-<pinref part="PAD3" gate="G$1" pin="P"/>
+<pinref part="PAD4" gate="G$1" pin="P"/>
 </segment>
 </net>
@@
 <wire x1="109.22" y1="12.7" x2="109.22" y2="7.62" width="0.1524" layer="91"/>
 <pinref part="R18" gate="G$1" pin="1"/>
-<pinref part="PAD4" gate="P" pin="P"/>
+<pinref part="PAD6" gate="P" pin="P"/>
 </segment>
 </net>
@@
 <pinref part="R3" gate="G$1" pin="1"/>
 <pinref part="R2" gate="G$1" pin="1"/>
-</segment>
-<segment>
-<pinref part="Q7" gate="G1" pin="B"/>
-<wire x1="170.18" y1="68.58" x2="175.26" y2="68.58" width="0.1524" layer="91"/>
+<pinref part="PAD8" gate="G$1" pin="P"/>
 </segment>
 </net>
@@
 <wire x1="114.3" y1="35.56" x2="160.02" y2="35.56" width="0.1524" layer="91"/>
 <wire x1="109.22" y1="50.8" x2="160.02" y2="50.8" width="0.1524" layer="91"/>
-<wire x1="160.02" y1="50.8" x2="172.72" y2="50.8" width="0.1524" layer="91"/>
+<wire x1="160.02" y1="50.8" x2="167.64" y2="50.8" width="0.1524" layer="91"/>
 <junction x="160.02" y="50.8"/>
+<pinref part="PAD1" gate="1" pin="P"/>
 <pinref part="PAD5" gate="1" pin="P"/>
-<pinref part="PAD1" gate="1" pin="P"/>
-<wire x1="53.34" y1="45.72" x2="53.34" y2="50.8" width="0.1524" layer="91"/>
-<junction x="53.34" y="50.8"/>
+<wire x1="167.64" y1="50.8" x2="172.72" y2="50.8" width="0.1524" layer="91"/>
+<wire x1="167.64" y1="45.72" x2="167.64" y2="50.8" width="0.1524" layer="91"/>
+<junction x="167.64" y="50.8"/>
 </segment>
 </net>
@@
 <wire x1="129.54" y1="154.94" x2="119.38" y2="154.94" width="0.1524" layer="91"/>
 <junction x="119.38" y="154.94"/>
-<pinref part="PAD6" gate="1" pin="P"/>
+<pinref part="PAD2" gate="1" pin="P"/>
 <wire x1="109.22" y1="154.94" x2="109.22" y2="157.48" width="0.1524" layer="91"/>
 </segment>
 </net>
+<net name="FBJ" class="0">
+<segment>
+<pinref part="Q7" gate="G1" pin="B"/>
+<wire x1="170.18" y1="68.58" x2="175.26" y2="68.58" width="0.1524" layer="91"/>
+<pinref part="PAD9" gate="G$1" pin="P"/>
+</segment>
+</net>

Commit message: Fixed board CNC errors, ready for cutting on othermill
Parts:
- R17: device rcl:R-US_0207/7 -> resistor:R-US_0309/12
Changed lines of the file:
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@@
 <part name="R11" library="rcl" library_urn="urn:adsk.eagle:library:334" deviceset="R-US_" device="0207/7" package3d_urn="urn:adsk.eagle:package:23493/1"/>
 <part name="R12" library="rcl" library_urn="urn:adsk.eagle:library:334" deviceset="R-US_" device="0207/7" package3d_urn="urn:adsk.eagle:package:23493/1"/>
-<part name="R17" library="rcl" library_urn="urn:adsk.eagle:library:334" deviceset="R-US_" device="0207/7" package3d_urn="urn:adsk.eagle:package:23493/1"/>
+<part name="R17" library="resistor" library_urn="urn:adsk.eagle:library:348" deviceset="R-US_" device="0309/12" package3d_urn="urn:adsk.eagle:package:26089/1"/>
 <part name="R18" library="rcl" library_urn="urn:adsk.eagle:library:334" deviceset="R-US_" device="0207/7" package3d_urn="urn:adsk.eagle:package:23493/1"/>
 <part name="C1" library="rcl" library_urn="urn:adsk.eagle:library:334" deviceset="CPOL-US" device="E2.5-7" package3d_urn="urn:adsk.eagle:package:23345/1"/>

Commit message: Minor updates to Motor Controller
Parts:
- added D7: 1N4148DO35-10, diode:1N4148DO35-10
Connections:
- removed net PWM: PAD6.P, R18.1
- new net N$2: D7.C, R18.1
- new net N$4: D7.A, PAD6.P
Other:
- moved on the sheet: PAD6
Changed lines of the file:
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@@
 <part name="PAD8" library="wirepad" library_urn="urn:adsk.eagle:library:412" deviceset="WIREPAD" device="2,54/1,1" package3d_urn="urn:adsk.eagle:package:30836/1"/>
 <part name="PAD9" library="wirepad" library_urn="urn:adsk.eagle:library:412" deviceset="WIREPAD" device="2,54/1,1" package3d_urn="urn:adsk.eagle:package:30836/1"/>
+<part name="D7" library="diode" library_urn="urn:adsk.eagle:library:210" deviceset="1N4148" device="DO35-10" package3d_urn="urn:adsk.eagle:package:43344/2"/>
 </parts>
 <sheets>
@@
 <instance part="PAD3" gate="G$1" x="101.6" y="109.22" rot="R180"/>
 <instance part="PAD4" gate="G$1" x="114.3" y="109.22"/>
-<instance part="PAD6" gate="P" x="109.22" y="5.08" rot="R90"/>
+<instance part="PAD6" gate="P" x="109.22" y="-5.08" rot="R90"/>
 <instance part="PAD1" gate="1" x="175.26" y="50.8" rot="R180"/>
 <instance part="PAD2" gate="1" x="109.22" y="160.02" rot="R270"/>
@@
 <instance part="PAD8" gate="G$1" x="-17.78" y="129.54"/>
 <instance part="PAD9" gate="G$1" x="177.8" y="68.58" rot="R180"/>
+<instance part="D7" gate="G$1" x="109.22" y="5.08" rot="R90"/>
 </instances>
 <busses>
@@
 <wire x1="-50.8" y1="121.92" x2="-50.8" y2="139.7" width="0.1524" layer="91"/>
 <pinref part="PAD7" gate="P" pin="P"/>
-</segment>
-</net>
-<net name="PWM" class="0">
-<segment>
-<wire x1="109.22" y1="12.7" x2="109.22" y2="7.62" width="0.1524" layer="91"/>
-<pinref part="R18" gate="G$1" pin="1"/>
-<pinref part="PAD6" gate="P" pin="P"/>
 </segment>
 </net>
@@
 </segment>
 </net>
+<net name="N$2" class="0">
+<segment>
+<pinref part="R18" gate="G$1" pin="1"/>
+<pinref part="D7" gate="G$1" pin="C"/>
+<wire x1="109.22" y1="12.7" x2="109.22" y2="7.62" width="0.1524" layer="91"/>
+</segment>
+</net>
+<net name="N$4" class="0">
+<segment>
+<pinref part="D7" gate="G$1" pin="A"/>
+<pinref part="PAD6" gate="P" pin="P"/>
+<wire x1="109.22" y1="2.54" x2="109.22" y2="-2.54" width="0.1524" layer="91"/>
+</segment>
+</net>
