File: Circuits/Boards/MotorControllerBoard/MotorBoard/MainBoard.brd (EAGLE design)
At the start: 124.4 x 87.3 mm, 59 parts, among them IC2 788TV, M1 IRFS7537PBF, M2 IRFS7537PBF, M3 IRFS7537PBF, M4 IRFS7537PBF, Q1 2N3904, Q2 2N3904, Q3 2N3904, Q4 2N3904, Q5 2N3904, Q6 2N3904, Q7 2N3904, Q8 2N3904

Commit message: Split off 22V & 5V circuits, shrunk motor controller and began adding second to single board
Parts:
- removed C1, C2, C3, C4, C5: (no value), rcl:E2,5-7
- removed IC1: (no value), ic-package:DIL08
- removed IC2: 788TV, linear:TO220V
- removed L1: (no value), eagle-ltspice:0207/10
- added D10, D11, D12, D8, D9: 1N4148DO35-10, diode:DO35-10
- added M5, M6, M7, M8: IRFS7537PBF, EagleCAD:D2PACK
- added PAD10, PAD11, PAD13, PAD16, PAD17: (no value), wirepad:2,54/1,1
- added PAD12: WIREPAD4,16O1,6, wirepad:4,16O1,6
- added PAD14, PAD18, PAD19, PAD20: (no value), wirepad:3,81/1,4
- added PAD15: (no value), wirepad:2,54/1,0
- added Q10, Q11, Q12, Q13, Q14, Q15, Q16, Q9: 2N3904, transistor-npn:TO92
- added R24, R25, R26, R27, R29: (no value), rcl:0207/7
- added R28: (no value), resistor:0207/7
- added R30, R31, R32, R33, R34: (no value), ptc-ntc:P660A
- PAD6: device wirepad:2,54/1,0 -> wirepad:2,54/1,1
- PAD8: value WIREPAD2,54/1,1 -> (none); device wirepad:2,54/1,1 -> wirepad:3,81/1,4
- PAD9: value WIREPAD2,54/1,1 -> WIREPAD4,16O1,6; device wirepad:2,54/1,1 -> wirepad:4,16O1,6
- R17: device resistor:0309/12 -> resistor:0207/7
- moved R14 184.7 mm to (-161.3, -2.54)
- moved R15 180.9 mm to (-139.7, -2.54), turned to 0 degrees
- moved R16 163.0 mm to (-118.1, -2.54)
- moved D6 118.8 mm to (-88.9, 26.7), turned to 0 degrees
- moved PAD8 112.3 mm to (121.9, 90.2), turned to 90 degrees
- moved R2 106.0 mm to (113.0, 31.8), turned to 180 degrees
- moved R3 104.5 mm to (-88.9, 11.4), turned to 0 degrees
- moved R5 102.4 mm to (-67.3, 11.4)
- moved R11 101.6 mm to (109.2, 34.3)
- moved Q2 98.0 mm to (111.8, 21.6), turned to 0 degrees
- moved R18 89.2 mm to (96.5, 21.6)
- moved R13 88.2 mm to (-45.7, 11.4)
- moved PAD7 87.5 mm to (88.9, 27.9), turned to 180 degrees
- moved Q8 86.4 mm to (104.1, 24.1), turned to 180 degrees
- moved D7 83.9 mm to (87.6, 24.1), turned to 180 degrees
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Connections:
- removed net FBJ: PAD9.1, Q7.2
- removed net N$1: PAD2.1, R19.1, R20.1, R21.1, R22.1, R23.1
- removed net N$12: IC1.7, L1.2, R15.1, R16.2
- removed net N$13: IC1.5, R13.1, R14.2
- removed net VG2: C2.+, D6.C, R13.2
- new net BB1: Q11.2, Q12.2, Q9.2, R3.2
- new net BF1: M7.1, Q11.1, R14.2, R16.1
- new net DIR1: D11.A, PAD15.1
- new net FB1: Q10.2, Q15.2, Q9.1, R5.1
- new net FF1: M5.1, Q10.1, R13.1, R15.2
- new net MN1: D10.C, D8.A, M7.3, M8.2, PAD12.1
- new net MP1: D6.A, D9.C, M5.3, M6.2, PAD9.1
- new net N$6: Q13.2, Q14.2, Q16.1, R26.2
- new net N$8: D11.C, R3.1
- new net VBAT: PAD1.1, PAD14.1, PAD2.1, PAD20.1, R19.1, R20.1, R21.1, R22.1, R23.1, R30.1, R31.1, R32.1, R33.1, R34.1
- new net VDD1: D6.C, D8.C, M5.2, M7.2, R30.2, R31.2, R32.2, R33.2, R34.2
- new net VG1: PAD17.1, R13.2, R14.1, R27.2, R28.2
- new net VSW1: PAD16.1, R26.1, R5.2
- net 0: now also D10.A, D9.A, M6.3, M8.3, PAD18.1, PAD19.1, PAD8.1, Q10.3, Q11.3, Q12.3, Q13.3, Q14.3, Q15.3, Q16.3, Q9.3, R15.1, R16.2, R24.2, R25.2; no longer C1.-, C2.-, C3.+, C4.-, C5.-, IC1.2, IC1.4, IC2.2, PAD1.1, R14.1
- net BB: now also Q3.2; no longer R5.1
- net FB: now also Q2.2, Q7.2; no longer PAD8.1, R3.1
- net N$10: now also D12.C, R29.1; no longer C3.-, IC1.3
- net N$11: now also D12.A, PAD13.1; no longer IC1.8, R16.1
- net N$3: now also M6.1, Q12.1, Q13.1, R25.1, R27.1; no longer Q2.2, R3.2
- net N$5: now also M8.1, Q14.1, Q15.1, R24.1, R28.1; no longer D6.A, IC1.1, L1.1
- net N$7: now also Q16.2, R29.2; no longer Q3.2, R5.2
- net VDD: no longer C1.+, C5.+, IC1.6, IC2.1, R12.2, R15.2, R17.2
- net VG: now also PAD11.1, R12.2, R17.2
- net VSW: now also PAD10.1; no longer C4.+, IC2.3
Routing:
- net 0: track 542.1 -> 185.8 mm
- net VDD: track 323.5 -> 100.9 mm
- net VSW: track 134.4 -> 8.89 mm
- net N$16: track 135.9 -> 38.6 mm
- net VBAT: track 0.00 -> 81.3 mm
- net N$1: track 71.1 -> 0.00 mm
- net VG2: track 66.0 -> 0.00 mm
- net VDD1: track 0.00 -> 66.0 mm
- net N$20: track 97.9 -> 57.3 mm
- net BF: track 74.9 -> 36.8 mm
- net N$12: track 36.8 -> 0.00 mm
- net BB: track 62.8 -> 31.1 mm
- net N$27: track 58.4 -> 34.3 mm
- net VG: track 5.08 -> 28.5 mm
- net DIR: track 25.4 -> 8.89 mm
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Other:
- board size 124.4 x 87.3 mm -> 127 x 101.3 mm

Commit message: Single board, two motor update
Parts:
- added PAD21, PAD22, PAD23, PAD24: (no value), wirepad:2,54/1,1
- R14, R15, R25: device rcl:0207/7 -> resistor:0207/7
- R16, R24: device rcl:0207/7 -> resistor:0207/12
- moved R15 201.5 mm to (34.3, 99.1)
- moved PAD15 200.7 mm to (36.8, 33.0)
- moved R14 196.5 mm to (29.2, 45.7), turned to 270 degrees
- moved R28 188.0 mm to (17.8, 40.6)
- moved Q13 186.5 mm to (21.6, 45.7)
- moved D10 183.5 mm to (14.0, 69.8), turned to 180 degrees
- moved R29 175.6 mm to (30.5, 26.7), turned to 180 degrees
- moved D11 168.6 mm to (31.8, 29.2)
- moved R16 161.8 mm to (31.8, 58.4), turned to 270 degrees
- moved PAD16 161.7 mm to (21.6, 30.5)
- moved Q14 161.5 mm to (14.0, 47.0), turned to 180 degrees
- moved PAD18 159.7 mm to (5.08, 86.4)
- moved D12 153.7 mm to (40.6, 31.8), turned to 90 degrees
- moved PAD17 148.2 mm to (36.8, 47.0)
- moved Q15 141.4 mm to (12.7, 36.8), turned to 180 degrees
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Connections:
- removed net BF1: M7.1, Q11.1, R14.2, R16.1
- new net BFF: PAD21.1, Q11.1, R14.2
- new net BFG: M7.1, PAD22.1, R16.1
- new net N$1: M8.1, PAD23.1, R24.1
- net N$5: now also PAD24.1; no longer M8.1, R24.1
Routing:
- net 0: track 185.8 -> 541.6 mm
- net VBAT: track 81.3 -> 422.5 mm
- net VDD1: track 66.0 -> 250.3 mm
- net VDD: track 100.9 -> 255.7 mm
- net FF1: track 0.00 -> 142.2 mm
- net N$3: track 0.00 -> 81.7 mm
- net FB1: track 0.00 -> 58.4 mm
- net MN1: track 0.00 -> 55.7 mm
- net MP1: track 0.00 -> 51.3 mm
- net VG1: track 0.00 -> 41.9 mm
- net N$6: track 0.00 -> 41.2 mm
- net BB1: track 0.00 -> 26.9 mm
- net N$5: track 0.00 -> 17.8 mm
- net BFF: track 0.00 -> 10.2 mm
- net N$7: track 0.00 -> 9.53 mm
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