File: Circuits/Boards/KiCAD/Motors/22VPowerBoard.kicad_pcb (KiCad board)
At the start: 2 copper layers, 30.5 x 25.4 mm, 13 parts, among them J1 Conn_01x01, J2 Conn_01x01, J3 Conn_01x01, U1 HCPL063

Commit message: Update KiCAD motor controller and Version 2 simulation
Parts:
- R3: value 16.5K -> 20K
Changed lines of the file:
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@@
     (links 21)
     (no_connects 2)
-    (area 101.344981 96.0926 134.695001 124.2174)
+    (area 104.064999 96.444999 134.695001 121.995001)
     (thickness 1.6)
     (drawings 4)
@@
   )
   (setup
-    (last_trace_width 1.27)
+    (last_trace_width 0.8128)
     (user_trace_width 0.1524)
     (user_trace_width 0.8128)
@@
     (pad_to_mask_clearance 0.2)
     (aux_axis_origin 0 0)
-    (visible_elements 7FFFFFFF)
+    (visible_elements 7FFFFFDF)
     (pcbplotparams
       (layerselection 0x01000_80000001)
@@
       (effects (font (size 1 1) (thickness 0.15)))
     )
-    (fp_text value 16.5K (at 1.27 2.31 180) (layer F.Fab)
+    (fp_text value 20K (at 1.27 2.31 180) (layer F.Fab)
       (effects (font (size 1 1) (thickness 0.15)))
     )
@@
   (segment (start 124.46 111.76) (end 129.54 111.76) (width 1.27) (layer Top) (net 3))
   (segment (start 124.46 111.76) (end 124.46 115.57) (width 1.27) (layer Top) (net 3))
-  (segment (start 111.76 100.33) (end 111.76 97.79) (width 1.27) (layer Top) (net 4) (status 400000))
-  (segment (start 121.92 97.79) (end 121.92 100.33) (width 1.27) (layer Top) (net 4) (status 800000))
+  (segment (start 111.76 100.33) (end 111.76 97.79) (width 1.27) (layer Top) (net 4))
+  (segment (start 121.92 97.79) (end 121.92 100.33) (width 1.27) (layer Top) (net 4))
   (segment (start 111.76 97.79) (end 121.92 97.79) (width 1.27) (layer Top) (net 4))
   (segment (start 111.76 104.14) (end 111.76 100.33) (width 1.27) (layer Top) (net 4) (status 20))
