File: Circuits/Boards/KiCAD/Motors/SingleMotorBoard.sch (KiCad schematic (older format))
At the start: 45 parts, among them M1 IRFS7537PBF, M2 IRFS7537PBF, M3 IRFS7537PBF, M4 IRFS7537PBF, Q1 2N3904, Q2 2N3904, Q3 2N3904, Q4 2N3904, Q5 2N3904, Q6 2N3904, Q7 2N3904, Q8 2N3904

Commit message: Update KiCAD motor controller and Version 2 simulation
Parts:
- removed D1, D2, D3, D4, D5, D7: 1N4148DO35-10, DIODE_DO35-10, symbol DIODE_1N4148DO35-10
- removed M1, M2, M3, M4: IRFS7537PBF, EAGLECAD_D2PACK, symbol EAGLECAD_IRFS7537PBF
- removed PAD1, PAD2, PAD5, PAD8: (no value), WIREPAD_3_81_1_4, symbol WIREPAD_3_81_1_4
- removed PAD10, PAD11, PAD6: (no value), WIREPAD_2_54_1_1, symbol WIREPAD_2_54_1_1
- removed PAD3, PAD4: WIREPAD4,16O1,6, WIREPAD_4_16O1_6, symbol WIREPAD_WIREPAD4_16O1_6
- removed PAD7: (no value), WIREPAD_2_54_1_0, symbol WIREPAD_2_54_1_0
- removed Q1, Q2, Q3, Q4, Q5, Q6, Q7, Q8: 2N3904, TRANSISTOR-NPN_TO92, symbol TRANSISTOR-NPN_2N3904
- removed R1, R10, R11, R12, R18, R2, R4, R6, R7, R8, R9: (no value), RCL_0207_7, symbol RCL_R-US_0207_7
- removed R17: (no value), RESISTOR_0207_7, symbol RESISTOR_R-US_0207_7
- removed R19, R20, R21, R22, R23: (no value), PTC-NTC_P660A, symbol PTC-NTC_PTC660A
- added D1, D2, D3, D4, D5, D6, D7, D8: 1N4007, Diodes_THT:D_5W_P5.08mm_Vertical_AnodeUp, symbol D
- added J1: Conn_01x05, Connectors_Molex:Molex_KK-6410-05_05x2.54mm_Straight, symbol Conn_01x05
- added J2, J3, J4, J5, J6, J7: Conn_01x01, Wire_Pads:SolderWirePad_single_2-5mmDrill, symbol Conn_01x01
- added Q1, Q2, Q3, Q4, Q5, Q6, Q7, Q8, Q9: 2N3904, TO_SOT_Packages_THT:TO-92_Inline_Wide, symbol Q_NPN_EBC
- added Q10, Q11, Q12, Q13: Q_NMOS_DGS, TO_SOT_Packages_SMD:TO-263-2, symbol Q_NMOS_GDS
- added R1, R10, R13, R15, R3, R4, R6, R7, R8, R9: 10K, Resistors_THT:R_Axial_DIN0207_L6.3mm_D2.5mm_P2.54mm_Vertical, symbol R
- added R11, R2, R5: 1K, Resistors_THT:R_Axial_DIN0207_L6.3mm_D2.5mm_P2.54mm_Vertical, symbol R
- added R12, R14: 1Meg, Resistors_THT:R_Axial_DIN0207_L6.3mm_D2.5mm_P2.54mm_Vertical, symbol R
- added TH1, TH2, TH3, TH4, TH5: Thermistor_PTC, Fuse_Holders_and_Fuses:Fuse_Littelfuse-LVR200, symbol Thermistor_PTC
Connections:
- net labels added: BBM, Dir, FBM, GND, MBB, MBF, MFB, MFF, Speed, iSpeed
- net labels removed: 0, BB, BF, DIR, FB, FF, MN, MP, N$16, N$19, N$2, N$20, N$23, N$27, N$4, VBAT, VDD
- wire segments 123 -> 100

Commit message: Fixed KiCAD motor controller
Parts:
- J1: footprint Connectors_Molex:Molex_KK-6410-05_05x2.54mm_Straight -> Connectors_JST:JST_VH_B5P-VH-B_5x3.96mm_Vertical
Changed lines of the file:
@@
 LIBS:contrib
 LIBS:valves
+LIBS:SingleMotorBoard-cache
 EELAYER 25 0
 EELAYER END
@@
 F 0 "J1" H 850 1400 50  0000 C CNN
 F 1 "Conn_01x05" H 850 800 50  0000 C CNN
-F 2 "Connectors_Molex:Molex_KK-6410-05_05x2.54mm_Straight" H 850 1100 50  0001 C CNN
+F 2 "Connectors_JST:JST_VH_B5P-VH-B_5x3.96mm_Vertical" H 850 1100 50  0001 C CNN
 F 3 "" H 850 1100 50  0001 C CNN
 	1    850  1100

Commit message: Rerouted motor controller for smaller size
Parts:
- J1: footprint Connectors_JST:JST_VH_B5P-VH-B_5x3.96mm_Vertical -> Connectors_JST:JST_XH_B05B-XH-A_05x2.50mm_Straight
Changed lines of the file:
@@
 F 0 "J1" H 850 1400 50  0000 C CNN
 F 1 "Conn_01x05" H 850 800 50  0000 C CNN
-F 2 "Connectors_JST:JST_VH_B5P-VH-B_5x3.96mm_Vertical" H 850 1100 50  0001 C CNN
+F 2 "Connectors_JST:JST_XH_B05B-XH-A_05x2.50mm_Straight" H 850 1100 50  0001 C CNN
 F 3 "" H 850 1100 50  0001 C CNN
 	1    850  1100
