File: Circuits/Boards/KiCAD/Motors/26VUnit.sch (KiCad schematic (older format))
At the start: 10 parts, among them U1 MC34063

Commit message: Fixed missing connections and routing
Parts:
- removed U1: MC34063, Housings_DIP:DIP-8_W7.62mm, symbol HCPL063
- added J17: MC34063, Housings_DIP:DIP-8_W7.62mm, symbol Conn_02x04_Counter_Clockwise
Connections:
- net labels removed: N$11
Other:
- moved on the sheet: C1, C2, C3, D17, L1, R31, R32, R33
