File: Circuits/Boards/KiCAD/Motors/MotorControlUnit.sch (KiCad schematic (older format))
At the start: 48 parts, among them J1 Conn_01x05, J2 Conn_01x01, J3 Conn_01x01, J4 Conn_01x01, J5 Conn_01x01, J6 Conn_01x01, J7 Conn_01x01, Q1 2N3904, Q10 Q_NMOS_DGS, Q11 Q_NMOS_DGS, Q12 Q_NMOS_DGS, Q13 Q_NMOS_DGS, Q2 2N3904, Q3 2N3904, Q4 2N3904, Q5 2N3904, Q6 2N3904, Q7 2N3904, Q8 2N3904, Q9 2N3904

Commit message: Added 26V and 5V units to the Dual motor controller board
Parts:
- removed TH1, TH2, TH3, TH4, TH5: Thermistor_PTC, Resistors_THT:R_Axial_DIN0207_L6.3mm_D2.5mm_P7.62mm_Horizontal, symbol Thermistor_PTC
- added F2, F3, F4, F5, F6: Polyfuse, Resistors_THT:R_Axial_DIN0207_L6.3mm_D2.5mm_P7.62mm_Horizontal, symbol Polyfuse
Connections:
- net labels added: DVG, DVSW, VFUSE
- net labels removed: VFuse
- wire segments 102 -> 106
Other:
- moved on the sheet: D10, D9

Commit message: Added drain resistors to gates
Parts:
- added C6, C7: 1200uF, Capacitors_THT:C_Disc_D12.0mm_W4.4mm_P7.75mm, symbol CP1
- added R35, R36, R37: 10K, Resistors_THT:R_Axial_DIN0207_L6.3mm_D2.5mm_P2.54mm_Vertical, symbol R
Connections:
- wire segments 106 -> 116
Other:
- moved on the sheet: Q15, Q21, R17, R22, R24, R26
